File: hardware/Eagle/Xmas_base_board.brd (EAGLE design)
At the start: 60 x 60 mm, 12 parts, among them CN1 MRUSB-2B-D14NI-S306_MRUSB-2B

Commit message: garber data upload
Other:
- board text added: "Rev 1.02"
- board text removed: "Rev 1.01"
Changed lines of the file:
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@@
 <drawing>
 <settings>
-<setting alwaysvectorfont="yes"/>
+<setting alwaysvectorfont="no"/>
 <setting verticaltext="up"/>
 </settings>
@@
 <text x="17.55" y="55.71" size="2.1844" layer="21">LED Christmas tree</text>
 <text x="48.26" y="3.81" size="1.778" layer="22" rot="MR0">NS-DIY-1001</text>
-<text x="48.26" y="1.27" size="1.778" layer="22" rot="MR0">Rev 1.01</text>
+<text x="48.26" y="1.27" size="1.778" layer="22" rot="MR0">Rev 1.02</text>
 <rectangle x1="38.84295" y1="55.11165" x2="39.14775" y2="55.14975" layer="200" rot="R180"/>
 <rectangle x1="38.72865" y1="55.14975" x2="39.14775" y2="55.18785" layer="200" rot="R180"/>
