File: hardware/Eagle/Xmas_A_board.brd (EAGLE design)
At the start: 60 x 118.9 mm, 32 parts

Commit message: garber data upload
Parts:
- moved R1 5.14 mm to (18.7, 43.2)
- moved C3 3.72 mm to (19.1, 33.0), turned to 0 degrees
- moved C1 3.70 mm to (40.1, 33.1)
- moved R5 1.15 mm to (40.6, 43.2)
- moved C2 0.97 mm to (46.0, 33.0)
Routing:
- net N$3: track 46.8 -> 51.6 mm
- net N$10: track 228.3 -> 230.9 mm
- net N$1: track 14.7 -> 15.9 mm
- net VCC: track 319.9 -> 320.9 mm
- net N$8: track 48.8 -> 49.7 mm
- net N$5: track 37.4 -> 38.1 mm
- net N$7: track 45.8 -> 45.2 mm
- net N$2: track 277.0 -> 277.5 mm
Other:
- board text added: "Rev 1.02"

Commit message: 抵抗の定数変更
Parts:
- added U$1, U$2: XMAS_POWER, xmas_p:XMAS_POWER
- R1, R3, R5: value 330 -> 1k
- R2, R4, R6: value 330 -> 100
Connections:
- net GND: now also U$1.P$1, U$1.P$2
- net VCC: now also U$2.P$1, U$2.P$2
Routing:
- net GND: track 101.7 -> 102.1 mm, vias 1 -> 0
- net VCC: vias 1 -> 0
Changed lines of the file:
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@@
 <setting verticaltext="up"/>
 </settings>
-<grid distance="50" unitdist="mil" unit="mil" style="lines" multiple="1" display="yes" altdistance="5" altunitdist="mil" altunit="mil"/>
+<grid distance="50" unitdist="mil" unit="mil" style="lines" multiple="1" display="no" altdistance="5" altunitdist="mil" altunit="mil"/>
 <layers>
 <layer number="1" name="Top" color="4" fill="1" visible="yes" active="yes"/>
@@
 <attribute name="VALUE" x="50.322690625" y="34.35471875" size="1.27" layer="27" ratio="10" rot="R300"/>
 </element>
-<element name="R2" library="rcl" library_urn="urn:adsk.eagle:library:334" package="0204/7" package3d_urn="urn:adsk.eagle:package:23498/2" value="330" x="14.986" y="28.321" smashed="yes" rot="R180">
+<element name="R2" library="rcl" library_urn="urn:adsk.eagle:library:334" package="0204/7" package3d_urn="urn:adsk.eagle:package:23498/2" value="100" x="14.986" y="28.321" smashed="yes" rot="R180">
 <attribute name="NAME" x="14.2875" y="29.77515" size="1.016" layer="25" ratio="10"/>
 <attribute name="POPULARITY" value="48" x="-2.794" y="70.231" size="1.778" layer="27" rot="R180" display="off"/>
@@
 <attribute name="VALUE" x="16.6116" y="28.8036" size="0.9906" layer="27" ratio="10" rot="R180"/>
 </element>
-<element name="R4" library="rcl" library_urn="urn:adsk.eagle:library:334" package="0204/7" package3d_urn="urn:adsk.eagle:package:23498/2" value="330" x="35.56" y="67.31" smashed="yes" rot="R90">
+<element name="R4" library="rcl" library_urn="urn:adsk.eagle:library:334" package="0204/7" package3d_urn="urn:adsk.eagle:package:23498/2" value="100" x="35.56" y="67.31" smashed="yes" rot="R90">
 <attribute name="NAME" x="34.3281" y="66.70675" size="1.016" layer="25" ratio="10" rot="R90"/>
 <attribute name="POPULARITY" value="48" x="77.47" y="95.25" size="1.778" layer="27" rot="R90" display="off"/>
@@
 <attribute name="VALUE" x="36.0426" y="65.6844" size="0.9906" layer="27" ratio="10" rot="R90"/>
 </element>
-<element name="R6" library="rcl" library_urn="urn:adsk.eagle:library:334" package="0204/7" package3d_urn="urn:adsk.eagle:package:23498/2" value="330" x="25.3365" y="74.3585" smashed="yes" rot="R90">
+<element name="R6" library="rcl" library_urn="urn:adsk.eagle:library:334" package="0204/7" package3d_urn="urn:adsk.eagle:package:23498/2" value="100" x="25.3365" y="74.3585" smashed="yes" rot="R90">
 <attribute name="NAME" x="24.0411" y="73.533" size="1.016" layer="25" ratio="10" rot="R90"/>
 <attribute name="POPULARITY" value="48" x="67.2465" y="112.4585" size="1.778" layer="27" rot="R90" display="off"/>
@@
 <attribute name="VALUE" x="25.8191" y="72.7329" size="0.9906" layer="27" ratio="10" rot="R90"/>
 </element>
-<element name="R1" library="rcl" library_urn="urn:adsk.eagle:library:334" package="0204/7" package3d_urn="urn:adsk.eagle:package:23498/2" value="330" x="18.669" y="43.18" smashed="yes" rot="R180">
+<element name="R1" library="rcl" library_urn="urn:adsk.eagle:library:334" package="0204/7" package3d_urn="urn:adsk.eagle:package:23498/2" value="1k" x="18.669" y="43.18" smashed="yes" rot="R180">
 <attribute name="NAME" x="17.907" y="44.50715" size="1.016" layer="25" ratio="10"/>
 <attribute name="POPULARITY" value="48" x="0.889" y="90.17" size="1.778" layer="27" rot="R180" display="off"/>
@@
 <attribute name="VALUE" x="20.2946" y="43.6626" size="0.9906" layer="27" ratio="10" rot="R180"/>
 </element>
-<element name="R3" library="rcl" library_urn="urn:adsk.eagle:library:334" package="0204/7" package3d_urn="urn:adsk.eagle:package:23498/2" value="330" x="44.196" y="28.3845" smashed="yes">
+<element name="R3" library="rcl" library_urn="urn:adsk.eagle:library:334" package="0204/7" package3d_urn="urn:adsk.eagle:package:23498/2" value="1k" x="44.196" y="28.3845" smashed="yes">
 <attribute name="NAME" x="43.59275" y="29.7434" size="1.016" layer="25" ratio="10"/>
 <attribute name="POPULARITY" value="48" x="72.136" y="-18.6055" size="1.778" layer="27" display="off"/>
@@
 <attribute name="VALUE" x="42.5704" y="27.9019" size="0.9906" layer="27" ratio="10"/>
 </element>
-<element name="R5" library="rcl" library_urn="urn:adsk.eagle:library:334" package="0204/7" package3d_urn="urn:adsk.eagle:package:23498/2" value="330" x="40.64" y="43.18" smashed="yes">
+<element name="R5" library="rcl" library_urn="urn:adsk.eagle:library:334" package="0204/7" package3d_urn="urn:adsk.eagle:package:23498/2" value="1k" x="40.64" y="43.18" smashed="yes">
 <attribute name="NAME" x="40.10025" y="44.4754" size="1.016" layer="25" ratio="10"/>
 <attribute name="POPULARITY" value="48" x="78.74" y="-3.81" size="1.778" layer="27" display="off"/>
@@
 <attribute name="VALUE" x="26.7996" y="118.2034" size="1.27" layer="27" ratio="10" rot="R180"/>
 </element>
+<element name="U$1" library="xmas_p" package="XMAS_POWER" value="XMAS_POWER" x="22.479" y="3.048" smashed="yes"/>
+<element name="U$2" library="xmas_p" package="XMAS_POWER" value="XMAS_POWER" x="37.465" y="3.048" smashed="yes"/>
 </elements>
 <signals>
@@
 <wire x1="48.006" y1="28.3845" x2="53.99535" y2="28.3845" width="0.4064" layer="1"/>
 <wire x1="53.99535" y1="28.3845" x2="54.61" y2="27.76985" width="0.4064" layer="1"/>
-<via x="37.465" y="3.429" extent="1-16" drill="0.35" diameter="3.302" shape="square"/>
 <wire x1="37.465" y1="3.429" x2="37.465" y2="24.13" width="1.016" layer="1"/>
 <wire x1="45.7835" y1="26.162" x2="48.006" y2="28.3845" width="1.016" layer="1"/>
@@
 <wire x1="41.4655" y1="88.5825" x2="41.266990625" y2="88.781009375" width="0.4064" layer="16"/>
 <wire x1="50.165" y1="39.751" x2="46.736" y2="43.18" width="0.4064" layer="16"/>
+<contactref element="U$2" pad="P$1"/>
+<contactref element="U$2" pad="P$2"/>
+<wire x1="37.465" y1="3.048" x2="37.465" y2="3.048" width="0" layer="19" extent="1-16"/>
+<wire x1="37.465" y1="3.429" x2="37.465" y2="3.048" width="0" layer="19" extent="1-1"/>
 </signal>
 <signal name="N$2">
@@
 <wire x1="25.654" y1="60.706" x2="22.86" y2="60.706" width="0.4064" layer="16"/>
 <wire x1="27.305" y1="82.20075" x2="27.305" y2="62.357" width="0.4064" layer="16"/>
-<via x="22.479" y="3.429" extent="1-16" drill="0.35" diameter="3.302" shape="square"/>
-<wire x1="22.479" y1="3.429" x2="22.479" y2="26.035" width="1.016" layer="1"/>
 <wire x1="30.099" y1="33.655" x2="30.099" y2="44.704" width="1.016" layer="1"/>
 <wire x1="30.099" y1="44.704" x2="35.56" y2="50.165" width="1.016" layer="1"/>
 <wire x1="35.56" y1="50.165" x2="35.687" y2="50.165" width="1.016" layer="1"/>
-<wire x1="22.479" y1="26.035" x2="30.099" y2="33.655" width="1.016" layer="1"/>
+<contactref element="U$1" pad="P$2"/>
+<wire x1="22.987" y1="26.543" x2="30.099" y2="33.655" width="1.016" layer="1"/>
+<contactref element="U$1" pad="P$1"/>
+<wire x1="22.479" y1="3.048" x2="22.479" y2="26.035" width="1.016" layer="1"/>
+<wire x1="22.479" y1="26.035" x2="22.987" y2="26.543" width="1.016" layer="1"/>
+<wire x1="22.479" y1="3.048" x2="22.479" y2="3.048" width="0" layer="19" extent="1-16"/>
 </signal>
 <signal name="N$1">
