File: hardware/Eagle/Xmas_B_board.brd (EAGLE design)
At the start: 60 x 118.9 mm, 30 parts

Commit message: garber data upload
Parts:
- moved R1 4.08 mm to (15.0, 40.9)
- moved C3 2.24 mm to (21.8, 31.5)
- moved C2 2.00 mm to (45.1, 31.4)
- moved C1 2.00 mm to (36.4, 31.5)
- moved R2 2.00 mm to (15.0, 26.3)
Routing:
- net N$1: track 14.7 -> 18.8 mm
- net N$2: track 255.0 -> 258.1 mm
- net N$8: track 60.5 -> 62.5 mm
- net N$6: track 36.4 -> 38.4 mm
- net N$5: track 31.4 -> 33.4 mm
- net N$3: track 79.4 -> 81.2 mm
- net N$7: track 45.8 -> 47.4 mm
- net VCC: track 289.5 -> 288.4 mm
Other:
- board text added: "Rev 1.02"

Commit message: 抵抗の定数変更
Parts:
- added U$1, U$2: XMAS_POWER, xmas_p:XMAS_POWER
- R1, R3, R5: value 330 -> 1k
- R2, R4, R6: value 330 -> 100
Connections:
- net GND: now also U$2.P$1, U$2.P$2
- net VCC: now also U$1.P$1, U$1.P$2
Routing:
- net VCC: vias 1 -> 0
- net GND: vias 1 -> 0
Changed lines of the file:
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@@
 <drawing>
 <settings>
-<setting alwaysvectorfont="yes"/>
+<setting alwaysvectorfont="no"/>
 <setting verticaltext="up"/>
 </settings>
@@
 <attribute name="VALUE" x="50.322690625" y="34.35471875" size="1.27" layer="27" ratio="10" rot="R300"/>
 </element>
-<element name="R2" library="rcl" library_urn="urn:adsk.eagle:library:334" package="0204/7" package3d_urn="urn:adsk.eagle:package:23498/2" value="330" x="14.986" y="26.321" smashed="yes" rot="R180">
+<element name="R2" library="rcl" library_urn="urn:adsk.eagle:library:334" package="0204/7" package3d_urn="urn:adsk.eagle:package:23498/2" value="100" x="14.986" y="26.321" smashed="yes" rot="R180">
 <attribute name="NAME" x="14.2875" y="27.77515" size="1.016" layer="25" ratio="10"/>
 <attribute name="POPULARITY" value="48" x="-2.794" y="68.231" size="1.778" layer="27" rot="R180" display="off"/>
@@
 <attribute name="VALUE" x="16.6116" y="26.8036" size="0.9906" layer="27" ratio="10" rot="R180"/>
 </element>
-<element name="R4" library="rcl" library_urn="urn:adsk.eagle:library:334" package="0204/7" package3d_urn="urn:adsk.eagle:package:23498/2" value="330" x="37.973" y="45.7835" smashed="yes">
+<element name="R4" library="rcl" library_urn="urn:adsk.eagle:library:334" package="0204/7" package3d_urn="urn:adsk.eagle:package:23498/2" value="100" x="37.973" y="45.7835" smashed="yes">
 <attribute name="NAME" x="37.36975" y="47.0154" size="1.016" layer="25" ratio="10"/>
 <attribute name="POPULARITY" value="48" x="65.913" y="3.8735" size="1.778" layer="27" display="off"/>
@@
 <attribute name="VALUE" x="36.3474" y="45.3009" size="0.9906" layer="27" ratio="10"/>
 </element>
-<element name="R6" library="rcl" library_urn="urn:adsk.eagle:library:334" package="0204/7" package3d_urn="urn:adsk.eagle:package:23498/2" value="330" x="25.3365" y="74.3585" smashed="yes" rot="R90">
+<element name="R6" library="rcl" library_urn="urn:adsk.eagle:library:334" package="0204/7" package3d_urn="urn:adsk.eagle:package:23498/2" value="100" x="25.3365" y="74.3585" smashed="yes" rot="R90">
 <attribute name="NAME" x="24.0411" y="73.533" size="1.016" layer="25" ratio="10" rot="R90"/>
 <attribute name="POPULARITY" value="48" x="67.2465" y="112.4585" size="1.778" layer="27" rot="R90" display="off"/>
@@
 <attribute name="VALUE" x="25.8191" y="72.7329" size="0.9906" layer="27" ratio="10" rot="R90"/>
 </element>
-<element name="R1" library="rcl" library_urn="urn:adsk.eagle:library:334" package="0204/7" package3d_urn="urn:adsk.eagle:package:23498/2" value="330" x="14.9545" y="40.9095" smashed="yes" rot="R180">
+<element name="R1" library="rcl" library_urn="urn:adsk.eagle:library:334" package="0204/7" package3d_urn="urn:adsk.eagle:package:23498/2" value="1k" x="14.9545" y="40.9095" smashed="yes" rot="R180">
 <attribute name="NAME" x="14.1925" y="42.23665" size="1.016" layer="25" ratio="10"/>
 <attribute name="POPULARITY" value="48" x="-2.8255" y="87.8995" size="1.778" layer="27" rot="R180" display="off"/>
@@
 <attribute name="VALUE" x="16.5801" y="41.3921" size="0.9906" layer="27" ratio="10" rot="R180"/>
 </element>
-<element name="R3" library="rcl" library_urn="urn:adsk.eagle:library:334" package="0204/7" package3d_urn="urn:adsk.eagle:package:23498/2" value="330" x="36.2585" y="63.3095" smashed="yes">
+<element name="R3" library="rcl" library_urn="urn:adsk.eagle:library:334" package="0204/7" package3d_urn="urn:adsk.eagle:package:23498/2" value="1k" x="36.2585" y="63.3095" smashed="yes">
 <attribute name="NAME" x="35.65525" y="64.6684" size="1.016" layer="25" ratio="10"/>
 <attribute name="POPULARITY" value="48" x="64.1985" y="16.3195" size="1.778" layer="27" display="off"/>
@@
 <attribute name="VALUE" x="34.6329" y="62.8269" size="0.9906" layer="27" ratio="10"/>
 </element>
-<element name="R5" library="rcl" library_urn="urn:adsk.eagle:library:334" package="0204/7" package3d_urn="urn:adsk.eagle:package:23498/2" value="330" x="22.733" y="55.753" smashed="yes" rot="R180">
+<element name="R5" library="rcl" library_urn="urn:adsk.eagle:library:334" package="0204/7" package3d_urn="urn:adsk.eagle:package:23498/2" value="1k" x="22.733" y="55.753" smashed="yes" rot="R180">
 <attribute name="NAME" x="23.27275" y="54.4576" size="1.016" layer="25" ratio="10" rot="R180"/>
 <attribute name="POPULARITY" value="48" x="-15.367" y="102.743" size="1.778" layer="27" rot="R180" display="off"/>
@@
 <attribute name="VALUE" x="19.6375" y="33.687" size="1.27" layer="27" ratio="10" rot="R180"/>
 </element>
+<element name="U$1" library="xmas_p" package="XMAS_POWER" value="XMAS_POWER" x="37.465" y="3.048" smashed="yes"/>
+<element name="U$2" library="xmas_p" package="XMAS_POWER" value="XMAS_POWER" x="22.479" y="3.048" smashed="yes"/>
 </elements>
 <signals>
@@
 <wire x1="22.135490625" y1="109.377240625" x2="23.129259375" y2="110.371009375" width="0.4064" layer="16"/>
 <wire x1="23.129259375" y1="110.371009375" x2="24.666725" y2="110.371009375" width="0.4064" layer="16"/>
-<via x="37.465" y="3.429" extent="1-16" drill="0.35" diameter="3.302" shape="square"/>
 <wire x1="37.465" y1="3.429" x2="37.465" y2="25.4" width="1.016" layer="1"/>
 <wire x1="40.0685" y1="63.3095" x2="41.148" y2="62.23" width="0.4064" layer="16"/>
@@
 <wire x1="41.41303125" y1="88.74125" x2="41.373271875" y2="88.781009375" width="0.4064" layer="16"/>
 <wire x1="42.70375" y1="88.74125" x2="43.561" y2="87.884" width="0.4064" layer="16"/>
+<contactref element="U$1" pad="P$2"/>
+<contactref element="U$1" pad="P$1"/>
+<wire x1="37.465" y1="3.048" x2="37.465" y2="3.048" width="0" layer="19" extent="1-16"/>
+<wire x1="37.465" y1="3.429" x2="37.465" y2="3.048" width="0" layer="19" extent="1-16"/>
 </signal>
 <signal name="N$2">
@@
 <contactref element="TR3" pad="E"/>
 <wire x1="22.86" y1="60.706" x2="22.86" y2="52.832" width="0.4064" layer="16"/>
-<via x="22.479" y="3.429" extent="1-16" drill="0.35" diameter="3.302" shape="square"/>
 <wire x1="26.035" y1="30.099" x2="26.035" y2="50.7365" width="1.016" layer="1"/>
 <wire x1="26.035" y1="50.7365" x2="23.9395" y2="52.832" width="1.016" layer="1"/>
@@
 <wire x1="28.448" y1="54.61" x2="28.448" y2="62.1665" width="0.508" layer="1"/>
 <wire x1="30.6705" y1="62.738" x2="31.6865" y2="61.722" width="0.508" layer="1"/>
+<contactref element="U$2" pad="P$1"/>
+<contactref element="U$2" pad="P$2"/>
+<wire x1="22.479" y1="3.048" x2="22.479" y2="3.429" width="0" layer="19" extent="1-1"/>
+<wire x1="22.479" y1="3.048" x2="22.479" y2="3.048" width="0" layer="19" extent="1-16"/>
 </signal>
 <signal name="N$1">
