File: hardware/Eagle/Xmas_B_board.sch (EAGLE design)
At the start: 30 parts

Commit message: 抵抗の定数変更
Parts:
- added U$1, U$2: XMAS_POWER, xmas_p:XMAS_POWER
- R1, R3, R5: value 330 -> 1k
- R2, R4, R6: value 330 -> 100
Connections:
- net GND: now also U$2.P$1, U$2.P$2
- net VCC: now also U$1.P$1, U$1.P$2
Other:
- moved on the sheet: C1, C2, C3, LED1, LED10, LED11, LED12, LED13, LED14, LED15, LED16, LED17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
